File: hw/VGMPlayer.kicad_sch (KiCad schematic)
At the start: 99 parts, among them J1 Micro_SD_Card, J2 EarPiece, P1 USB_C_Receptacle_16P, P2 SWD, P3 BATT, P5 ICSP, P6 CODEC, Q1 AO3401A, Q2 AO3401A, Q3 2N7002, Q4 2N7002, U1 RP2040, U2 W25QxxJVZP, U3 LP5907MFX-3.3, U4 WM8978, U5 MCP73831-OT, U6 PIC16F1503-IMG, U7 LP5907MFX-3.3, Y1 12MHz

Commit message: V4 hardware
Parts:
- removed C14, C23: 1u, BZ_Capacitor:C_0603, symbol BZ_Passive:C
- removed C17, C19, C21, C27: 100n, BZ_Capacitor:C_0402, symbol BZ_Passive:C
- removed C24: DNP, BZ_Capacitor:C_0402, symbol BZ_Passive:C
- removed JP1: Jumper-NC, BZ_Misc:Jumper-Solder, symbol BZ_Misc:Jumper-NC
- removed JP2, JP3: Jumper-NO, BZ_Misc:Jumper-Solder, symbol BZ_Misc:Jumper-NO
- removed R13: 1K, BZ_Resistor:R_0402, symbol BZ_Passive:R
- removed U3: LP5907MFX-3.3, BZ_Standard_IC:SOT-23-5, symbol BZ_TI:LP5907MFX
- C18, C20, C22, C25, C26: value 10u -> 4.7u
Connections:
- net 3V3: now also C25.1, FB1.2
- net VIN: now also C22.1, C33.1, Q2.3 (D), U4.26 (SPKVDD), U7.1 (IN), U7.3 (EN); no longer FB1.2
- net BEEP: no longer names the net of U4.19 (AUXL)
- net VDDA: no longer names the net of C20.1, U4.31 (AVDD)
- net VDDA: now also FB1.1; no longer C25.1
- no-connect marks 22 -> 24
Other:
- moved on the sheet: C18, C20, C22, C25, C26, C28, C29, C30, FB1, J2, P6, R14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

Commit message: V4 hardware
Parts:
- removed C30: 1u, BZ_Capacitor:C_0603, symbol BZ_Passive:C
- added C20: 1u, BZ_Capacitor:C_0603, symbol BZ_Passive:C
- added C21: 100n, BZ_Capacitor:C_0402, symbol BZ_Passive:C
- added U4: MAX9890BETA, BZ_Standard_IC:TDFN-8-1EP_3x3x0.65P_EP2.3x1.5, symbol BZ_Maxim:MAX9890BETA
- S1: value M -> U
- S2: value P -> B
- S3: value U -> D
- S4: value D -> P
- S5: value RESET -> F; footprint BZ_Switch:SW-PUSH_4x3x2H -> VGMPlayer:MultiButton
- renumbered C25 to C15, C18 to C16, C20 to C17, C22 to C18, C26 to C19, C28 to C22, C29 to C23, C16 to C24, C31 to C25, C33 to C26, C34 to C27, C35 to C28, C32 to C29, C36 to C30, U4 to U3
Connections:
- net GND: now also C20.2, C21.2, U4.5 (GND), U4.9 (GND)
- net JACK_DET: now also U1.38 (GPIO26_ADC0)
- net OUTEN: now reaches U1.31 (GPIO20)
- net OUTEN: now also U4.2 (~{SHDN})
- net at U3.29 (ROUT1): now also U4.7 (INR); no longer C22.1
- net at U3.30 (LOUT1): now also U4.3 (INL); no longer C23.1
- net AVDD: now reaches C17.1, FB1.1, U3.31 (AVDD)
- net AVDD: now also C20.1, U4.1 (VCC)
- new net: C22.1, U4.6 (OUTR)
- new net: C23.1, U4.4 (OUTL)
- new net: C21.1, U4.8 (CEXT)
- no-connect marks 24 -> 22
Other:
- moved on the sheet: C15, C16, C17, C18, C19, C22, C23, D2, FB1, J2, P6, R14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

Commit message: V4 hardware send for JLC
Parts:
- removed C27: DNP, BZ_Capacitor:C_0402, symbol BZ_Passive:C
- removed Q2: AO3401A, BZ_Standard_IC:SOT-23-3, symbol BZ_FET:MOS_P_GSD
- removed R20: 100K, BZ_Resistor:R_0402, symbol BZ_Passive:R
- removed U7: LP5907MFX-3.3, BZ_Standard_IC:SOT-23-5, symbol BZ_TI:LP5907MFX
- added C29: 4.7u, BZ_Capacitor:C_0603, symbol BZ_Passive:C
- added R13: 10K, BZ_Resistor:R_0402, symbol BZ_Passive:R
- added U7: XC6220B331MR, BZ_Standard_IC:SOT-23-5, symbol BZ_Torex:XC6220B331MR
- C26: value 1u -> 4.7u; PN (none) -> GRM188R61A106KE69D
- R21: value 10K -> 100K
- renumbered C15 to C14, C16 to C15, C17 to C16, C18 to C17, C20 to C18, C21 to C19, C19 to C20, C22 to C21, C23 to C22, C24 to C23, C25 to C24, C28 to C25, C29 to C27, C30 to C28
Connections:
- net 3V3: now also C26.1, C29.1, U7.5 (VOUT); no longer C25.1
- net AVDD: now also C17.1, U3.26 (SPKVDD)
- net GND: now also R21.2, C29.2, R13.1, U7.2 (VSS)
- net OUTEN: now also R13.2
- net VIN: no longer C17.1, C26.1, U3.26 (SPKVDD)
- net VRAW: now also C25.1, U7.1 (VIN)
- net at R21.1: now also U6.7 (RC2), U7.3 (CE)
Other:
- moved on the sheet: C25, P5, R21

Commit message: MCP73831->MCP83832
Parts:
- U5: value MCP73831-OT -> MCP73832-OT; symbol BZ_Microchip:MCP73831-OT -> BZ_Microchip:MCP73832-OT
Changed lines of the file:
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@@
     (pin "1")
   )
-  (symbol (lib_id "BZ_Microchip:MCP73831-OT") (at 43.18 46.99 0) (unit 1)
+  (symbol (lib_id "BZ_Microchip:MCP73832-OT") (at 43.18 46.99 0) (unit 1)
     (in_bom yes) (on_board yes)
     (property "Reference" "U5" (id 0) (at 39.37 40.64 0)
       (effects (font (size 1.016 1.016)))
     )
-    (property "Value" "MCP73831-OT" (id 1) (at 43.18 50.8 0)
+    (property "Value" "MCP73832-OT" (id 1) (at 43.18 50.8 0)
       (effects (font (size 1.016 1.016)))
     )
@@
     )
     (path "/00000000-0000-0000-0000-0000615b852d"
-      (reference "U5") (unit 1) (value "MCP73831-OT") (footprint "BZ_Standard_IC:SOT-23-5")
+      (reference "U5") (unit 1) (value "MCP73832-OT") (footprint "BZ_Standard_IC:SOT-23-5")
     )
     (path "/00000000-0000-0000-0000-000060931bcc"

Commit message: Update switch names
Parts:
- S1: value U -> NW
- S2: value B -> SE
- S3: value D -> SW
- S4: value P -> PLAY
- S5: value F -> NE
Changed lines of the file:
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@@
       (effects (font (size 1.016 1.016)))
     )
-    (property "Value" "D" (id 1) (at 45.72 58.42 0)
+    (property "Value" "SW" (id 1) (at 45.72 58.42 0)
       (effects (font (size 1.016 1.016)) (justify left))
     )
@@
       (effects (font (size 1.016 1.016)))
     )
-    (property "Value" "U" (id 1) (at 45.72 55.88 0)
+    (property "Value" "NW" (id 1) (at 45.72 55.88 0)
       (effects (font (size 1.016 1.016)) (justify left))
     )
@@
       (effects (font (size 1.016 1.016)))
     )
-    (property "Value" "B" (id 1) (at 45.72 66.04 0)
+    (property "Value" "SE" (id 1) (at 45.72 66.04 0)
       (effects (font (size 1.016 1.016)) (justify left))
     )
@@
     (pin "12")
     (pin "13")
+    (pin "14")
+    (pin "15")
     (pin "16")
     (pin "17")
@@
       (effects (font (size 1.016 1.016)))
     )
-    (property "Value" "F" (id 1) (at 45.72 63.5 0)
+    (property "Value" "NE" (id 1) (at 45.72 63.5 0)
       (effects (font (size 1.016 1.016)) (justify left))
     )
@@
       (effects (font (size 1.016 1.016)))
     )
-    (property "Value" "P" (id 1) (at 45.72 60.96 0)
+    (property "Value" "PLAY" (id 1) (at 45.72 60.96 0)
       (effects (font (size 1.016 1.016)) (justify left))
     )
@@
     )
     (path "/00000000-0000-0000-0000-0000606e50c2"
-      (reference "S1") (unit 1) (value "U") (footprint "VGMPlayer:MultiButton")
+      (reference "S1") (unit 1) (value "NW") (footprint "VGMPlayer:MultiButton")
     )
     (path "/00000000-0000-0000-0000-000060860be8"
-      (reference "S2") (unit 1) (value "B") (footprint "VGMPlayer:MultiButton")
+      (reference "S2") (unit 1) (value "SE") (footprint "VGMPlayer:MultiButton")
     )
     (path "/00000000-0000-0000-0000-0000606e358e"
-      (reference "S3") (unit 1) (value "D") (footprint "VGMPlayer:MultiButton")
+      (reference "S3") (unit 1) (value "SW") (footprint "VGMPlayer:MultiButton")
     )
     (path "/00000000-0000-0000-0000-000061b88515"
-      (reference "S4") (unit 1) (value "P") (footprint "VGMPlayer:MultiButton")
+      (reference "S4") (unit 1) (value "PLAY") (footprint "VGMPlayer:MultiButton")
     )
     (path "/00000000-0000-0000-0000-0000613792ff"
-      (reference "S5") (unit 1) (value "F") (footprint "VGMPlayer:MultiButton")
+      (reference "S5") (unit 1) (value "NE") (footprint "VGMPlayer:MultiButton")
     )
     (path "/00000000-0000-0000-0000-000060986baa"
